File: display-unit-PCB/display-unit.kicad_pcb (KiCad board)
At the start: 2 copper layers, 3 parts, among them J1 RJ45_LED_Shielded, J2 Display, J3 ESP32 38-Pin

Commit message: trying to migrate
Parts:
- added J4: SD_Card, Connector_PinSocket_2.54mm:PinSocket_1x04_P2.54mm_Vertical, F.Cu at (220.0, 66.7)
- added J5: RTC, Connector_PinSocket_2.54mm:PinSocket_1x04_P2.54mm_Vertical, F.Cu at (73.5, 45.0)
- added U1: MAX3485, Package_DIP:DIP-8_W7.62mm, F.Cu at (100.0, 66.4)
- moved J2 154.3 mm to (198.0, 57.1)
- moved J1 73.1 mm to (98.2, 94.5), turned to 180 degrees
- moved J3 57.9 mm to (140.7, 70.3), turned to 180 degrees
Connections:
- J1 pad 1: Net-(J2-14) -> Net-(J1-Pad1)
- J1 pad 2: Net-(J3-Pin_22) -> Net-(J3-Pin_20)
- J1 pad 3: Net-(J2-Pin_2) -> Net-(U1-B)
- J1 pad 4: Net-(J2-Pin_11) -> Net-(J3-Pin_20)
- J1 pad 5: Net-(J2-Pin_2) -> Net-(U1-A)
- J1 pad 6: Net-(J2-Pin_12) -> Net-(J3-Pin_20)
- J1 pad 7: Net-(J2-Pin_2) -> unconnected-(J1-Pad7)
- J1 pad 8: Net-(J2-Pin_7) -> unconnected-(J1-Pad8)
- J2 pad D/C: Net-(J2-Pin_5) -> unconnected-(J2-Pin_5-PadD/C)
- J2 pad LED: Net-(J2-14) -> unconnected-(J2-Pin_7-PadLED)
- J2 pad SCK: Net-(J2-Pin_7) -> Net-(J2-14)
- J2 pad T_CLK: Net-(J2-Pin_7) -> Net-(J2-14)
- J3 pad 14: Net-(J3-Pin_22) -> unconnected-(J3-Pin_22-Pad14)
- J3 pad 18: Net-(J2-Pin_7) -> Net-(J2-14)
- J3 pad 21: unconnected-(J3-Pin_2-Pad21) -> Net-(J5-Pin_2)
- J3 pad 22: unconnected-(J3-3.3-Pad22) -> Net-(J5-Pin_1)
- J3 pad 33: unconnected-(J3-Pin_27-Pad33) -> Net-(J3-Pin_27)
- J3 pad 5: Net-(J2-Pin_5) -> unconnected-(J3-Pin_6-Pad5)
- J3 pad 5V: Net-(J2-14) -> Net-(J1-Pad1)
- J3 pad RX: unconnected-(J3-3.3-PadRX) -> Net-(U1-R)
- J3 pad TX: unconnected-(J3-Pin_2-PadTX) -> Net-(U1-D)
Routing:
- net Net-(J2-14): track 95.1 -> 0.00 mm
- net Net-(J2-Pin_11): track 66.3 -> 0.00 mm
- net Net-(J2-Pin_10): track 62.1 -> 0.00 mm
- net Net-(J2-Pin_7): track 61.0 -> 0.00 mm
- net Net-(J2-Pin_12): track 55.8 -> 0.00 mm
- net Net-(J2-Pin_5): track 29.3 -> 0.00 mm
- net Net-(J2-Pin_4): track 29.3 -> 0.00 mm
- net Net-(J2-Pin_3): track 29.3 -> 0.00 mm
- net Net-(J2-Pin_2): track 0.61 -> 0.00 mm
